File: power.sch (KiCad schematic (older format))
At the start: 14 parts, among them U201 TPS54331DDAR

Commit message: Layout
Parts:
- 3.3V201: footprint (none) -> TestPoint:TestPoint_Pad_D1.5mm
- D201: footprint (none) -> Diode_SMD:D_SOD-123
- U201: footprint (none) -> VsReality_Footprints:Texas_Instruments-DDAR-PDSO-G8-12_2011-F-0
Connections:
- net GND: now also R202.2; no longer C204.2
- net at C203.1, U201.6 (COMP): now also C204.1; no longer R202.1
- new net: C204.2, R202.1
Other:
- moved on the sheet: C204, R202
Changed lines of the file:
@@
 F 0 "U201" H 4975 3515 50  0000 C CNN
 F 1 "TPS54331DDAR" H 4975 3424 50  0000 C CNN
-F 2 "" H 4750 3150 50  0001 C CNN
+F 2 "VsReality_Footprints:Texas_Instruments-DDAR-PDSO-G8-12_2011-F-0" H 4750 3150 50  0001 C CNN
 F 3 "" H 4750 3150 50  0001 C CNN
 	1    4850 3100
 	1    0    0    -1
 $EndComp
-Text GLabel 3100 2950 0    50   Input ~ 0
-BACK_IN
-Wire Wire Line
-	3150 2950 3150 3150
-Connection ~ 3150 2950
-Wire Wire Line
-	3150 2950 3100 2950
 $Comp
 L power:GND #PWR0203
@@
 U 1 1 6090A6A0
 P 7850 3050
+AR Path="/608F63EA/6090A6A0" Ref="3.3V201"  Part="1"
+AR Path="/6090A6A0" Ref="3.3V201"  Part="1"
 F 0 "3.3V201" H 7898 3096 50  0000 L CNN
 F 1 "TestPoint_Small" H 7898 3005 50  0000 L CNN
-F 2 "" H 8050 3050 50  0001 C CNN
+F 2 "TestPoint:TestPoint_Pad_D1.5mm" H 8050 3050 50  0001 C CNN
 F 3 "~" H 8050 3050 50  0001 C CNN
 	1    7850 3050
@@
 F 0 "D201" V 6104 3220 50  0000 L CNN
 F 1 "B5819W" V 6195 3220 50  0000 L CNN
-F 2 "" V 6150 3150 50  0001 C CNN
+F 2 "Diode_SMD:D_SOD-123" V 6150 3150 50  0001 C CNN
 F 3 "~" V 6150 3150 50  0001 C CNN
 	1    6150 3150
@@
 	4550 3300 4400 3300
 $Comp
-L Device:C_Small C204
-U 1 1 6091E757
-P 4000 3600
-F 0 "C204" H 4092 3646 50  0000 L CNN
-F 1 "1nF" H 4092 3555 50  0000 L CNN
-F 2 "Capacitor_SMD:C_0402_1005Metric" H 4000 3600 50  0001 C CNN
-F 3 "~" H 4000 3600 50  0001 C CNN
-F 4 "C1523" H 4000 3600 50  0001 C CNN "LCSC Part #"
-	1    4000 3600
-	1    0    0    -1
-$EndComp
-$Comp
 L Device:C_Small C203
 U 1 1 6091EC9C
@@
 $EndComp
 Wire Wire Line
-	3150 2950 4550 2950
-Wire Wire Line
 	3150 3750 3600 3750
 $Comp
 L Device:R_Small R202
 U 1 1 6092124E
-P 4000 3350
-F 0 "R202" H 4059 3396 50  0000 L CNN
-F 1 "30K" H 4059 3305 50  0000 L CNN
-F 2 "Resistor_SMD:R_0603_1608Metric" H 4000 3350 50  0001 C CNN
-F 3 "~" H 4000 3350 50  0001 C CNN
-F 4 "C22984" H 4000 3350 50  0001 C CNN "LCSC Part #"
-	1    4000 3350
-	1    0    0    -1
-$EndComp
-Wire Wire Line
-	4000 3450 4000 3500
+P 4000 3600
+F 0 "R202" H 4059 3646 50  0000 L CNN
+F 1 "30K" H 4059 3555 50  0000 L CNN
+F 2 "Resistor_SMD:R_0603_1608Metric" H 4000 3600 50  0001 C CNN
+F 3 "~" H 4000 3600 50  0001 C CNN
+F 4 "C22984" H 4000 3600 50  0001 C CNN "LCSC Part #"
+	1    4000 3600
+	1    0    0    -1
+$EndComp
 Wire Wire Line
 	4000 3700 4000 3750
@@
 Text Notes 3600 3900 0    50   ~ 0
 10nF=>4ms slow start
+Wire Wire Line
+	3150 2950 4550 2950
+Wire Wire Line
+	3150 2950 3100 2950
+Connection ~ 3150 2950
+Wire Wire Line
+	3150 2950 3150 3150
+Text GLabel 3100 2950 0    50   Input ~ 0
+BACK_IN
+$Comp
+L Device:C_Small C204
+U 1 1 6091E757
+P 4000 3350
+F 0 "C204" H 4092 3396 50  0000 L CNN
+F 1 "1nF" H 4092 3305 50  0000 L CNN
+F 2 "Capacitor_SMD:C_0402_1005Metric" H 4000 3350 50  0001 C CNN
+F 3 "~" H 4000 3350 50  0001 C CNN
+F 4 "C1523" H 4000 3350 50  0001 C CNN "LCSC Part #"
+	1    4000 3350
+	1    0    0    -1
+$EndComp
+Wire Wire Line
+	4000 3450 4000 3500
 $EndSCHEMATC

Commit message: Additional changes
Parts:
- D201: LCSC Part # (none) -> C8598
- U201: LCSC Part # (none) -> C90761
Changed lines of the file:
@@
 F 2 "VsReality_Footprints:Texas_Instruments-DDAR-PDSO-G8-12_2011-F-0" H 4750 3150 50  0001 C CNN
 F 3 "" H 4750 3150 50  0001 C CNN
+F 4 "C90761" H 4850 3100 50  0001 C CNN "LCSC Part #"
 	1    4850 3100
 	1    0    0    -1
@@
 F 2 "Diode_SMD:D_SOD-123" V 6150 3150 50  0001 C CNN
 F 3 "~" V 6150 3150 50  0001 C CNN
+F 4 "C8598" H 6150 3150 50  0001 C CNN "LCSC Part #"
 	1    6150 3150
 	0    1    1    0

Commit message: Change footprint for a comonent
Parts:
- U201: footprint VsReality_Footprints:Texas_Instruments-DDAR-PDSO-G8-12_2011-F-0 -> Package_SO:HSOP-8-1EP_3.9x4.9mm_P1.27mm_EP2.41x3.1mm_ThermalVias
Changed lines of the file:
@@
 F 0 "U201" H 4975 3515 50  0000 C CNN
 F 1 "TPS54331DDAR" H 4975 3424 50  0000 C CNN
-F 2 "VsReality_Footprints:Texas_Instruments-DDAR-PDSO-G8-12_2011-F-0" H 4750 3150 50  0001 C CNN
+F 2 "Package_SO:HSOP-8-1EP_3.9x4.9mm_P1.27mm_EP2.41x3.1mm_ThermalVias" H 4750 3150 50  0001 C CNN
 F 3 "" H 4750 3150 50  0001 C CNN
 F 4 "C90761" H 4850 3100 50  0001 C CNN "LCSC Part #"
