File: smart_motor_controller.sch (KiCad schematic (older format))
At the start: 42 parts, among them J10 USB_B_Micro, J101 Breakout, J102 I2C_CONN, J103 CAN_CONN, J104 Debug, J9 Input 12V, Q101 FDD6685, SW102 SW_NRST, SW103 SW_NRST, U2 STM32F405RGT6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

Commit message: Change in FDD6685
Parts:
- Q101: footprint Package_TO_SOT_SMD:TO-252-2 -> VsReality_Footprints:FDD6685
Changed lines of the file:
@@
 F 0 "Q101" V 1492 1500 50  0000 C CNN
 F 1 "FDD6685" V 1401 1500 50  0000 C CNN
-F 2 "Package_TO_SOT_SMD:TO-252-2" H 1350 1425 50  0001 L CIN
+F 2 "VsReality_Footprints:FDD6685" H 1350 1425 50  0001 L CIN
 F 3 "https://www.onsemi.com/pdf/datasheet/fdd6685-d.pdf" H 1150 1500 50  0001 L CNN
 F 4 "C10866" H 1150 1500 50  0001 C CNN "LCSC Part #"
