File: brushed_motors_and_encoders.kicad_sch (KiCad schematic)
At the start: 23 parts, among them J301 M0_CONN, J302 M1_CONN, J303 M2_CONN, J304 M3_CONN, J309 External encoders power, J310 Encoder Commector, U301 DRV8870DDA, U302 DRV8870DDA, U303 DRV8870DDA, U304 DRV8870DDA

Commit message: Updated gedber files
Parts:
- J310: LCSC Part # (none) -> C213462
Changed lines of the file:
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@@
+      (effects (font (size 1.27 1.27)) hide)
+    )
+    (property "LCSC Part #" "C213462" (at 44.45 127 0)
       (effects (font (size 1.27 1.27)) hide)
     )
