File: brushed_motors_and_encoders.kicad_sch (KiCad schematic)
At the start: 23 parts, among them J301 M0_CONN, J302 M1_CONN, J303 M2_CONN, J304 M3_CONN, J309 External encoders power, J310 Encoder Commector, U301 DRV8870DDA, U302 DRV8870DDA, U303 DRV8870DDA, U304 DRV8870DDA

Commit message: Initial changes
Parts:
- removed D301: B5819W, Diode_SMD:D_SOD-123, symbol Device:D_Schottky_Small
- removed J302: M1_CONN, VsReality_Footprints:Ningbo_Kangnex_Elec_WJ128V_5_0_2P, symbol Connector:Screw_Terminal_01x02
- removed J303: M2_CONN, VsReality_Footprints:Ningbo_Kangnex_Elec_WJ128V_5_0_2P, symbol Connector:Screw_Terminal_01x02
- removed J304: M3_CONN, VsReality_Footprints:Ningbo_Kangnex_Elec_WJ128V_5_0_2P, symbol Connector:Screw_Terminal_01x02
- removed J309: External encoders power, Connector_PinHeader_2.54mm:PinHeader_1x02_P2.54mm_Vertical, symbol smart_motor_controller-rescue:Conn_01x02_Male-Connector
- removed J310: Encoder Commector, VsReality_Footprints:Encoder_PinHeader_4x04_P2.54mm_Vertical, symbol smart_motor_controller-rescue:EncoderPinHeaderConnector_04-VsReality_Symbols
- removed R304: 0.15, Resistor_SMD:R_0603_1608Metric, symbol Device:R_Small
- removed U301, U302, U303, U304: DRV8870DDA, Package_SO:Texas_HTSOP-8-1EP_3.9x4.9mm_P1.27mm_EP2.95x4.9mm_Mask2.4x3.1mm_ThermalVias, symbol Driver_Motor:DRV8870DDA
- added C302, C311, C321, C331: 100n, Capacitor_SMD:C_0603_1608Metric, symbol Device:C_Small
- added C304, C306, C314, C316, C324, C326, C334, C336: 1u, Capacitor_SMD:C_0603_1608Metric, symbol Device:C_Small
- added C305, C315, C325, C335: 47n, Capacitor_SMD:C_0603_1608Metric, symbol Device:C_Small
- added J311, J321, J331: M0_CONN, VsReality_Footprints:Ningbo_Kangnex_Elec_WJ128V_5_0_2P, symbol Connector:Screw_Terminal_01x02
- added R311, R321, R331: 10K, Resistor_SMD:R_0603_1608Metric, symbol Device:R_Small
- added R312, R313, R322, R323, R332, R333: 330, Resistor_SMD:R_0603_1608Metric, symbol Device:R_Small
- added U301, U311, U321, U331: DRV8873S, VsReality_Footprints:HTSSOP-24_L7.8-W4.4-P0.65-LS6.4-TL-EP, symbol VsReality_Symbols:DRV8873S
- R301: value 0.15 -> 10K; LCSC Part # C45879 -> (none)
- R302, R303: value 0.15 -> 330; LCSC Part # C45879 -> (none)
- renumbered C302 to C303, C303 to C312, C304 to C313, C305 to C322, C306 to C323, C307 to C332, C308 to C333
Connections:
- net +3V3: now also R301.1, R311.1, R321.1, R331.1
- net GND: now also C302.1, C304.2, C311.1, C314.2, C321.1, C324.2, C331.1, C334.2, R312.2, R313.2, R322.2, R323.2, R332.2, R333.2, U301.16 (SRC), U301.17 (SRC), U301.24 (GND), U301.25 (EP), U311.16 (SRC), U311.17 (SRC), U311.24 (GND), U311.25 (EP), U321.16 (SRC), U321.17 (SRC), U321.24 (GND), U321.25 (EP), U331.16 (SRC), U331.17 (SRC), U331.24 (GND), U331.25 (EP); no longer R301.2
- net VMOTORS: now also C302.2, C306.1, C311.2, C316.1, C321.2, C326.1, C331.2, C336.1, U301.13 (VM), U301.20 (VM), U311.13 (VM), U311.20 (VM), U321.13 (VM), U321.20 (VM), U331.13 (VM), U331.20 (VM)
- net M0_IPROPI2: now reaches R303.1
- net M0_IPROPI2: now also U301.12 (IPROPI2)
- net M0_IPROPI1: now reaches R302.1
- net M0_IPROPI1: now also U301.10 (IPROPI1)
- net at J301.1 (Pin_1): now also U301.18 (OUT1), U301.19 (OUT1)
- net at J301.2 (Pin_2): now also U301.14 (OUT2), U301.15 (OUT2)
- new net: C324.1, U321.1 (DVDD)
- new net: C336.2, U331.21 (VCP)
- new net: C335.1, U331.22 (CPH)
- new net: C335.2, U331.23 (CPL)
- new net: C326.2, U321.21 (VCP)
- new net: C314.1, U311.1 (DVDD)
- new net: J321.2 (Pin_2), U321.14 (OUT2), U321.15 (OUT2)
- new net: J321.1 (Pin_1), U321.18 (OUT1), U321.19 (OUT1)
- new net: C325.1, U321.22 (CPH)
- new net: C325.2, U321.23 (CPL)
- new net: J331.1 (Pin_1), U331.18 (OUT1), U331.19 (OUT1)
- new net: J331.2 (Pin_2), U331.14 (OUT2), U331.15 (OUT2)
- new net: C334.1, U331.1 (DVDD)
- new net: C304.1, U301.1 (DVDD)
- new net: C306.2, U301.21 (VCP)
- new net: C315.1, U311.22 (CPH)
- new net: C315.2, U311.23 (CPL)
- new net: C316.2, U311.21 (VCP)
- new net: C305.1, U301.22 (CPH)
- new net: C305.2, U301.23 (CPL)
- new net: J311.1 (Pin_1), U311.18 (OUT1), U311.19 (OUT1)
- new net: J311.2 (Pin_2), U311.14 (OUT2), U311.15 (OUT2)
- new net M0_DISABLE: U301.9 (DISABLE)
- new net M0_EN: U301.7 (EN/IN1)
- new net M0_PH: U301.8 (PH/IN2)
- new net M0_nFAULT: R301.2, U301.2 (nFAULT)
- new net M0_nSCS: U301.6 (nSCS)
- new net M0_nSLEEP: U301.11 (nSLEEP)
- new net M1_DISABLE: U311.9 (DISABLE)
- new net M1_EN: U311.7 (EN/IN1)
- new net M1_IPROPI1: R312.1, U311.10 (IPROPI1)
- new net M1_IPROPI2: R313.1, U311.12 (IPROPI2)
- new net M1_PH: U311.8 (PH/IN2)
- new net M1_nFAULT: R311.2, U311.2 (nFAULT)
- new net M1_nSCS: U311.6 (nSCS)
- new net M1_nSLEEP: U311.11 (nSLEEP)
- new net M2_DISABLE: U321.9 (DISABLE)
- new net M2_EN: U321.7 (EN/IN1)
- new net M2_IPROPI1: R322.1, U321.10 (IPROPI1)
- new net M2_IPROPI2: R323.1, U321.12 (IPROPI2)
- new net M2_PH: U321.8 (PH/IN2)
- new net M2_nFAULT: R321.2, U321.2 (nFAULT)
- new net M2_nSCS: U321.6 (nSCS)
- new net M2_nSLEEP: U321.11 (nSLEEP)
- new net M3_DISABLE: U331.9 (DISABLE)
- new net M3_EN: U331.7 (EN/IN1)
- new net M3_IPROPI1: R332.1, U331.10 (IPROPI1)
- new net M3_IPROPI2: R333.1, U331.12 (IPROPI2)
- new net M3_PH: U331.8 (PH/IN2)
- new net M3_nFAULT: R331.2, U331.2 (nFAULT)
- new net M3_nSCS: U331.6 (nSCS)
- new net M3_nSLEEP: U331.11 (nSLEEP)
- new net M_SCLK: U301.5 (SCLK), U311.5 (SCLK), U321.5 (SCLK), U331.5 (SCLK)
- new net M_SDI: U301.4 (SDI), U311.4 (SDI), U321.4 (SDI), U331.4 (SDI)
- new net M_SDO: U301.3 (SDO), U311.3 (SDO), U321.3 (SDO), U331.3 (SDO)
Other:
- note added: "Motor 0"
- note added: "Motor 1"
- note added: "Motor 2"
- note added: "Motor 3"
- note removed: "I = 3.3/(10*R)"
- moved on the sheet: C301, C312, C313, C322, C323, C332, C333, J301

Commit message: Add USB sensing and power management components to the schematic
- Introduced a junction for USB sensing at coordinates (173.99, 64.77).
- Added multiple wires connecting various components to the new junction.
- Created a global label "USB_SENSE" for the USB sensing functionality.
- Updated references for power components to a new numbering scheme (#PWR0501 to #PWR0509).
- Added resistors R505 and R506 with specified values and footprints.
- Included power symbols for +5V and GND with appropriate references and properties.
- Ensured all new components are included in the BOM and marked for simulation.
Parts:
- added C310, C311, C324, C325: 1u, Capacitor_SMD:C_0603_1608Metric, symbol Device:C_Small
- R303: value 330 -> 100
- R304: renamed from R313; value 330 -> 100
- R309: renamed from R333; value 330 -> 100
- R310: renamed from R323; value 330 -> 100
- renumbered C304 to C301, C314 to C302, C305 to C303, C315 to C304, C306 to C305, C316 to C306, C311 to C307, C312 to C308, C313 to C309, C301 to C312, C302 to C313, C303 to C314, C334 to C315, C335 to C316, C324 to C317, C325 to C318, C336 to C319, C326 to C320, C331 to C321, C332 to C322, C333 to C323, C321 to C326, C322 to C327, C323 to C328, J311 to J302, J331 to J303, J321 to J304, R311 to R302, R302 to R305, R312 to R306, R331 to R307, R321 to R308, R332 to R311, R322 to R312, U311 to U302, U331 to U303, U321 to U304
Connections:
- net GND: now also C310.1, C311.1, C324.1, C325.1; no longer R303.2, R304.2, R309.2, R310.2
- net M0_IPROPI1: no longer names the net of R305.1, U301.10 (IPROPI1)
- net M0_IPROPI1: now also R303.2, U301.12 (IPROPI2), C310.2
- net M0_IPROPI2 renamed M0_IPROPI
- net M0_IPROPI: no longer U301.12 (IPROPI2)
- net M1_IPROPI1: no longer names the net of R306.1, U302.10 (IPROPI1)
- net M1_IPROPI1: now also R304.2, U302.12 (IPROPI2), C311.2
- net M1_IPROPI2 renamed M1_IPROPI
- net M1_IPROPI: no longer U302.12 (IPROPI2)
- net M2_IPROPI1: no longer names the net of R312.1, U304.10 (IPROPI1)
- net M2_IPROPI1: now also R310.2, U304.12 (IPROPI2), C325.2
- net M2_IPROPI2 renamed M2_IPROPI
- net M2_IPROPI: no longer U304.12 (IPROPI2)
- net M3_IPROPI1: no longer names the net of R311.1, U303.10 (IPROPI1)
- net M3_IPROPI1: now also R309.2, U303.12 (IPROPI2), C324.2
- net M3_IPROPI2 renamed M3_IPROPI
- net M3_IPROPI: no longer U303.12 (IPROPI2)
Other:
- moved on the sheet: R303, R304, R305, R306, R309, R310, R311, R312
