File: power.kicad_sch (KiCad schematic)
At the start: 18 parts, among them U201 TPS54331DDAR

Commit message: Edge of the bpard
Parts:
- H1, H2, H3, H4: footprint MountingHole:MountingHole_2.7mm_M2.5_Pad -> MountingHole:MountingHole_3.2mm_M3_DIN965_Pad
Changed lines of the file:
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@@
       (effects (font (size 1.27 1.27)) (justify left) hide)
     )
-    (property "Footprint" "MountingHole:MountingHole_2.7mm_M2.5_Pad" (at 248.92 91.44 0)
+    (property "Footprint" "MountingHole:MountingHole_3.2mm_M3_DIN965_Pad" (at 248.92 91.44 0)
       (effects (font (size 1.27 1.27)) hide)
     )
@@
       (effects (font (size 1.27 1.27)) (justify left) hide)
     )
-    (property "Footprint" "MountingHole:MountingHole_2.7mm_M2.5_Pad" (at 248.92 81.28 0)
+    (property "Footprint" "MountingHole:MountingHole_3.2mm_M3_DIN965_Pad" (at 248.92 81.28 0)
       (effects (font (size 1.27 1.27)) hide)
     )
@@
       (effects (font (size 1.27 1.27)) (justify left) hide)
     )
-    (property "Footprint" "MountingHole:MountingHole_2.7mm_M2.5_Pad" (at 248.92 76.2 0)
+    (property "Footprint" "MountingHole:MountingHole_3.2mm_M3_DIN965_Pad" (at 248.92 76.2 0)
       (effects (font (size 1.27 1.27)) hide)
     )
@@
       (effects (font (size 1.27 1.27)) (justify left) hide)
     )
-    (property "Footprint" "MountingHole:MountingHole_2.7mm_M2.5_Pad" (at 248.92 86.36 0)
+    (property "Footprint" "MountingHole:MountingHole_3.2mm_M3_DIN965_Pad" (at 248.92 86.36 0)
       (effects (font (size 1.27 1.27)) hide)
     )

Commit message: Change components to 0603
Parts:
- C201, C204: footprint Capacitor_SMD:C_0402_1005Metric -> Capacitor_SMD:C_0603_1608Metric
- C206, C207: footprint Capacitor_SMD:C_1206_3216Metric -> Capacitor_SMD:C_0603_1608Metric
- R201, R203: footprint Resistor_SMD:R_0402_1005Metric -> Resistor_SMD:R_0603_1608Metric
Changed lines of the file:
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@@
       (effects (font (size 1.27 1.27)) (justify left))
     )
-    (property "Footprint" "Capacitor_SMD:C_0402_1005Metric" (at 144.78 72.39 0)
+    (property "Footprint" "Capacitor_SMD:C_0603_1608Metric" (at 144.78 72.39 0)
       (effects (font (size 1.27 1.27)) hide)
     )
@@
       (effects (font (size 1.27 1.27)) (justify left))
     )
-    (property "Footprint" "Resistor_SMD:R_0402_1005Metric" (at 191.77 82.55 0)
+    (property "Footprint" "Resistor_SMD:R_0603_1608Metric" (at 191.77 82.55 0)
       (effects (font (size 1.27 1.27)) hide)
     )
@@
       (effects (font (size 1.27 1.27)) (justify left))
     )
-    (property "Footprint" "Resistor_SMD:R_0402_1005Metric" (at 191.77 90.17 0)
+    (property "Footprint" "Resistor_SMD:R_0603_1608Metric" (at 191.77 90.17 0)
       (effects (font (size 1.27 1.27)) hide)
     )
@@
       (effects (font (size 1.27 1.27)) (justify left))
     )
-    (property "Footprint" "Capacitor_SMD:C_0402_1005Metric" (at 101.6 85.09 0)
+    (property "Footprint" "Capacitor_SMD:C_0603_1608Metric" (at 101.6 85.09 0)
       (effects (font (size 1.27 1.27)) hide)
     )
@@
       (effects (font (size 1.27 1.27)) (justify left))
     )
-    (property "Footprint" "Capacitor_SMD:C_1206_3216Metric" (at 172.72 82.55 0)
+    (property "Footprint" "Capacitor_SMD:C_0603_1608Metric" (at 172.72 82.55 0)
       (effects (font (size 1.27 1.27)) hide)
     )
@@
       (effects (font (size 1.27 1.27)) (justify left))
     )
-    (property "Footprint" "Capacitor_SMD:C_1206_3216Metric" (at 181.61 82.55 0)
-      (effects (font (size 1.27 1.27)) hide)
-    )
+    (property "Footprint" "Capacitor_SMD:C_0603_1608Metric" (at 181.61 82.55 0)
+      (effects (font (size 1.27 1.27)) hide)
+    )

Commit message: Updated gedber files
Parts:
- C201: LCSC Part # C1525 -> C694249
- C203: LCSC Part # C57112 -> C915831
- C204: LCSC Part # C1523 -> C340644
- C206, C207: LCSC Part # C96123 -> C140782
- L201: LCSC Part # C139506 -> C351099
- R201: LCSC Part # C25744 -> C116677
- R203: LCSC Part # C25890 -> C269710
Changed lines of the file:
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@@
       (effects (font (size 1.27 1.27)) hide)
     )
-    (property "LCSC Part #" "C1525" (at 144.78 72.39 0)
+    (property "LCSC Part #" "C694249" (at 144.78 72.39 0)
       (effects (font (size 1.27 1.27)) hide)
     )
@@
       (effects (font (size 1.27 1.27)) hide)
     )
-    (property "LCSC Part #" "C139506" (at 167.64 77.47 0)
+    (property "LCSC Part #" "C351099" (at 167.64 77.47 0)
       (effects (font (size 1.27 1.27)) hide)
     )
@@
       (effects (font (size 1.27 1.27)) hide)
     )
-    (property "LCSC Part #" "C25744" (at 191.77 82.55 0)
+    (property "LCSC Part #" "C116677" (at 191.77 82.55 0)
       (effects (font (size 1.27 1.27)) hide)
     )
@@
       (effects (font (size 1.27 1.27)) hide)
     )
-    (property "LCSC Part #" "C25890" (at 191.77 90.17 0)
+    (property "LCSC Part #" "C269710" (at 191.77 90.17 0)
       (effects (font (size 1.27 1.27)) hide)
     )
@@
       (effects (font (size 1.27 1.27)) hide)
     )
-    (property "LCSC Part #" "C1523" (at 101.6 85.09 0)
+    (property "LCSC Part #" "C340644" (at 101.6 85.09 0)
       (effects (font (size 1.27 1.27)) hide)
     )
@@
       (effects (font (size 1.27 1.27)) hide)
     )
-    (property "LCSC Part #" "C57112" (at 91.44 91.44 0)
+    (property "LCSC Part #" "C915831" (at 91.44 91.44 0)
       (effects (font (size 1.27 1.27)) hide)
     )
@@
       (effects (font (size 1.27 1.27)) hide)
     )
-    (property "LCSC Part #" "C96123" (at 172.72 82.55 0)
+    (property "LCSC Part #" "C140782" (at 172.72 82.55 0)
       (effects (font (size 1.27 1.27)) hide)
     )
@@
       (effects (font (size 1.27 1.27)) hide)
     )
-    (property "LCSC Part #" "C96123" (at 181.61 82.55 0)
-      (effects (font (size 1.27 1.27)) hide)
-    )
+    (property "LCSC Part #" "C140782" (at 181.61 82.55 0)
+      (effects (font (size 1.27 1.27)) hide)
+    )

Commit message: Add CLAUDE.md for repository guidance and design documentation
- Introduced CLAUDE.md to provide an overview of the Kinisi smart motor controller board design.
- Included details on editing design files, fabrication workflow for JLCPCB, and revision management.
- Documented companion repositories for firmware and client libraries.
Parts:
- C203: LCSC Part # C915831 -> C57112
- C205: LCSC Part # C27920 -> C1322360
- renumbered H1 to H201, H2 to H202, H3 to H203, H4 to H204
