File: usb.kicad_sch (KiCad schematic)
At the start: 7 parts, among them J501 USB_C_Receptacle_USB2.0_16P, U501 USBLC6-2SC6

Commit message: Add USB sensing and power management components to the schematic
- Introduced a junction for USB sensing at coordinates (173.99, 64.77).
- Added multiple wires connecting various components to the new junction.
- Created a global label "USB_SENSE" for the USB sensing functionality.
- Updated references for power components to a new numbering scheme (#PWR0501 to #PWR0509).
- Added resistors R505 and R506 with specified values and footprints.
- Included power symbols for +5V and GND with appropriate references and properties.
- Ensured all new components are included in the BOM and marked for simulation.
Parts:
- added R505: 4K7, Resistor_SMD:R_0603_1608Metric, symbol Device:R_Small
- added R506: 10K, Resistor_SMD:R_0603_1608Metric, symbol Device:R_Small
- renumbered TP2 to TP501
Connections:
- net +5V: now also R505.2
- net GND: now also R506.1
- new net USB_SENSE: R505.1, R506.2
