File: IMU.kicad_sch (KiCad schematic)
At the start: 3 parts, among them U2 BMI088

Commit message: Add USB sensing and power management components to the schematic
- Introduced a junction for USB sensing at coordinates (173.99, 64.77).
- Added multiple wires connecting various components to the new junction.
- Created a global label "USB_SENSE" for the USB sensing functionality.
- Updated references for power components to a new numbering scheme (#PWR0501 to #PWR0509).
- Added resistors R505 and R506 with specified values and footprints.
- Included power symbols for +5V and GND with appropriate references and properties.
- Ensured all new components are included in the BOM and marked for simulation.
Parts:
- added C603: 10nf, Capacitor_SMD:C_0603_1608Metric, symbol Device:C_Small
- added R601, R602: 4k7, Resistor_SMD:R_0603_1608Metric, symbol Device:R_Small
- added U602: TMP102xxDRL, Package_TO_SOT_SMD:SOT-563, symbol Sensor_Temperature:TMP102xxDRL
- renumbered U2 to U601
Connections:
- net +3V3: now also C603.1, R601.1, R602.1, U602.5 (V+)
- net GND: now also C603.2, U602.2 (GND), U602.4 (ADD0)
- new net SENSOR_SCL: R601.2, U602.1 (SCL)
- new net SENSOR_SDA: R602.2, U602.6 (SDA)
- no-connect marks 0 -> 1
Other:
- note removed: "BMI088"
- moved on the sheet: C601, C602, U601

Commit message: Implement structure for code changes tracking
Parts:
- added C604: 100nf, Capacitor_SMD:C_0603_1608Metric, symbol Device:C_Small
- added U603: FM24C64B, Package_SO:SOIC-8_3.9x4.9mm_P1.27mm, symbol Memory_NVRAM:FM24C64B
Connections:
- net IMU_INT3_GYRO is gone; now on an unnamed net: U601.12 (INT3)
- net +3V3: now also C604.2, U603.8 (VDD)
- net GND: now also C604.1, U603.1 (A0), U603.2 (A1), U603.3 (A2), U603.4 (VSS), U603.7 (WP)
- net SENSOR_SCL: now also U603.6 (SCL)
- net SENSOR_SDA: now also U603.5 (SDA)
- net IMU_INT1_ACCEL: no longer names the net of U601.16 (INT1)
- net IMU_INT2_ACCEL renamed IMU_INT_ACCEL
- net IMU_INT4_GYRO renamed IMU_INT_GYRO
Other:
- note added: "Memory"
- note added: "https://www.bosch-sensortec.com/media/boschsensortec/downloads/application_notes_1/bst-mis-an006.pdf?utm_source=chatgpt.com"
